File: PCB/HDR camera controller/HDR camera controller.brd (EAGLE design)
At the start: 58 x 48 mm, 63 parts, among them IC1 USBLC6-4, IC10 RS422-SO8, IC11 RS422-SO8, IC12 USBLC6-4, IC14 741G157, IC2 RS422-SO8, IC3 RS422-SO8, IC4 RS422-SO8, IC6 FT232RL, IC7 74HC00D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

Commit message: PCB V1 manufacture
Parts:
- C11: value 100uF -> 47uF
Connections:
- net LINE_OUT_2: now also IC13.11; no longer IC13.28
Routing:
- net LINE_OUT_2: track 0.00 -> 35.7 mm, vias 0 -> 2
- net ENC_A: track 78.8 -> 83.6 mm
- net GND: track 495.3 -> 498.5 mm
- net HW_TRIG_SEL: track 23.7 -> 25.9 mm
- net ENC_B: track 92.1 -> 94.1 mm
- net HW_TRIG_TTL: track 56.4 -> 57.5 mm
- net LINE_IN_1: track 34.5 -> 35.5 mm
- net MISO: track 6.81 -> 7.46 mm
- added copper zone on layer 1, net GND
- added copper zone on layer 16, net GND
Other:
- outline, holes or cut-outs redrawn
- board text added: "HDR line cam controller V1"

Commit message: Timed trigger WIP
Connections:
- net B renamed L3
- net B+ renamed L3+
- net B- renamed L3-
- net G renamed L2
- net G+ renamed L2+
- net G- renamed L2-
- net R renamed L1
- net R+ renamed L1+
- net R- renamed L1-
Changed lines of the file:
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@@
 <wire x1="27.94" y1="46.355" x2="27.94" y2="44.9834" width="0.4064" layer="1"/>
 </signal>
-<signal name="R">
+<signal name="L1">
 <contactref element="IC7" pad="3"/>
 <contactref element="IC9" pad="3"/>
@@
 <wire x1="21.59" y1="33.02" x2="22.86" y2="33.02" width="0.4064" layer="1"/>
 </signal>
-<signal name="G">
+<signal name="L2">
 <contactref element="IC7" pad="6"/>
 <contactref element="IC10" pad="3"/>
@@
 <wire x1="19.05" y1="39.37" x2="22.86" y2="43.18" width="0.4064" layer="1"/>
 </signal>
-<signal name="B">
+<signal name="L3">
 <contactref element="IC7" pad="8"/>
 <contactref element="IC11" pad="3"/>
@@
 <wire x1="40.255" y1="35.625" x2="40.255" y2="37.015" width="0.4064" layer="1"/>
 </signal>
-<signal name="R+">
+<signal name="L1+">
 <contactref element="IC9" pad="6"/>
 <contactref element="LIGHT" pad="1"/>
@@
 <wire x1="5.715" y1="22.86" x2="2.54" y2="22.86" width="0.4064" layer="1"/>
 </signal>
-<signal name="R-">
+<signal name="L1-">
 <contactref element="IC9" pad="5"/>
 <contactref element="LIGHT" pad="2"/>
@@
 <wire x1="7.62" y1="28.829" x2="9.906" y2="31.115" width="0.4064" layer="1"/>
 </signal>
-<signal name="G+">
+<signal name="L2+">
 <contactref element="IC10" pad="6"/>
 <contactref element="LIGHT" pad="3"/>
@@
 <wire x1="7.62" y1="36.195" x2="7.62" y2="26.67" width="0.4064" layer="16"/>
 </signal>
-<signal name="G-">
+<signal name="L2-">
 <contactref element="IC10" pad="5"/>
 <contactref element="LIGHT" pad="4"/>
@@
 <wire x1="6.35" y1="36.83" x2="6.35" y2="27.305" width="0.4064" layer="16"/>
 </signal>
-<signal name="B+">
+<signal name="L3+">
 <contactref element="IC11" pad="6"/>
 <contactref element="LIGHT" pad="5"/>
@@
 <wire x1="3.81" y1="36.83" x2="8.89" y2="41.91" width="0.4064" layer="16"/>
 </signal>
-<signal name="B-">
+<signal name="L3-">
 <contactref element="IC11" pad="5"/>
 <contactref element="LIGHT" pad="6"/>

Commit message: tweaks
Connections:
- net RGB_IN renamed L_IN
- net RGB_SEL0 renamed L_SEL0
- net RGB_SEL1 renamed L_SEL1
Changed lines of the file:
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@@
 <wire x1="21.5646" y1="38.862" x2="21.59" y2="38.8366" width="0.4064" layer="1"/>
 </signal>
-<signal name="RGB_IN">
+<signal name="L_IN">
 <contactref element="IC7" pad="13"/>
 <contactref element="IC7" pad="12"/>
@@
 <wire x1="29.21" y1="20.193" x2="29.21" y2="29.21" width="0.4064" layer="16"/>
 </signal>
-<signal name="RGB_SEL0">
+<signal name="L_SEL0">
 <contactref element="IC8" pad="2"/>
 <contactref element="IC13" pad="23"/>
@@
 <wire x1="39.751" y1="28.194" x2="41.021" y2="26.924" width="0.4064" layer="16"/>
 </signal>
-<signal name="RGB_SEL1">
+<signal name="L_SEL1">
 <contactref element="IC8" pad="3"/>
 <contactref element="IC13" pad="24"/>
