File: PCB/HDR camera controller/HDR camera controller.sch (EAGLE design)
At the start: 63 parts, among them IC1 USBLC6-4, IC10 RS422-SO8, IC11 RS422-SO8, IC12 USBLC6-4, IC14 741G157, IC2 RS422-SO8, IC3 RS422-SO8, IC4 RS422-SO8, IC6 FT232RL, IC7 74HC00D, IC8 74HC139D, IC9 RS422-SO8, Q1 16MHz

Commit message: PCB V1 manufacture
Parts:
- C11: value 100uF -> 47uF; MPN (none) -> SC1E476M6L005VR
- FS1: MPN (none) -> SM010-60
- IC1, IC12: MPN (none) -> USBLC6
- IC14: MPN (none) -> 74LVC1G157GV.125
- IC7: MPN (none) -> SN74HC00DR
- IC8: MPN (none) -> SN74HC139DR
- Q1: MPN (none) -> 3225-16M-SR
- S1: MPN (none) -> A6S-6102-H
Connections:
- net LINE_OUT_2: now also IC13IC.PD7(AIN1/PCINT23); no longer IC13IC.PC5(ADC5/SCL/PCINT13)
Changed lines of the file:
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@@
 </classes>
 <parts>
-<part name="IC1" library="custom ICs" deviceset="USBLC6-4" device="" package3d_urn="urn:adsk.eagle:package:30993/1"/>
+<part name="IC1" library="custom ICs" deviceset="USBLC6-4" device="" package3d_urn="urn:adsk.eagle:package:30993/1">
+<attribute name="MPN" value="USBLC6"/>
+</part>
 <part name="C1" library="rcl" library_urn="urn:adsk.eagle:library:334" deviceset="C-EU" device="C0805" package3d_urn="urn:adsk.eagle:package:23617/2" value="100nF"/>
 <part name="R1" library="rcl" library_urn="urn:adsk.eagle:library:334" deviceset="R-EU_" device="R0805" package3d_urn="urn:adsk.eagle:package:23553/2" value="120R"/>
@@
 <part name="GND9" library="supply1" library_urn="urn:adsk.eagle:library:371" deviceset="GND" device=""/>
 <part name="GND10" library="supply1" library_urn="urn:adsk.eagle:library:371" deviceset="GND" device=""/>
-<part name="IC7" library="74xx-eu" library_urn="urn:adsk.eagle:library:85" deviceset="74*00" device="D" package3d_urn="urn:adsk.eagle:package:1010/2" technology="HC"/>
-<part name="IC8" library="74xx-eu" library_urn="urn:adsk.eagle:library:85" deviceset="74*139" device="D" package3d_urn="urn:adsk.eagle:package:2010/1" technology="HC"/>
+<part name="IC7" library="74xx-eu" library_urn="urn:adsk.eagle:library:85" deviceset="74*00" device="D" package3d_urn="urn:adsk.eagle:package:1010/2" technology="HC">
+<attribute name="MPN" value="SN74HC00DR"/>
+</part>
+<part name="IC8" library="74xx-eu" library_urn="urn:adsk.eagle:library:85" deviceset="74*139" device="D" package3d_urn="urn:adsk.eagle:package:2010/1" technology="HC">
+<attribute name="MPN" value="SN74HC139DR"/>
+</part>
 <part name="GND11" library="supply1" library_urn="urn:adsk.eagle:library:371" deviceset="GND" device=""/>
 <part name="GND12" library="supply1" library_urn="urn:adsk.eagle:library:371" deviceset="GND" device=""/>
-<part name="FS1" library="custom general" deviceset="POLYFUSE" device="_1210"/>
+<part name="FS1" library="custom general" deviceset="POLYFUSE" device="_1210">
+<attribute name="MPN" value="SM010-60"/>
+</part>
 <part name="C7" library="rcl" library_urn="urn:adsk.eagle:library:334" deviceset="C-EU" device="C0805" package3d_urn="urn:adsk.eagle:package:23617/2" value="100nF"/>
 <part name="C8" library="rcl" library_urn="urn:adsk.eagle:library:334" deviceset="C-EU" device="C0805" package3d_urn="urn:adsk.eagle:package:23617/2" value="100nF"/>
@@
 <part name="GND13" library="supply1" library_urn="urn:adsk.eagle:library:371" deviceset="GND" device=""/>
 <part name="GND14" library="supply1" library_urn="urn:adsk.eagle:library:371" deviceset="GND" device=""/>
-<part name="C11" library="rcl" library_urn="urn:adsk.eagle:library:334" deviceset="CPOL-EU" device="153CLV-0605" package3d_urn="urn:adsk.eagle:package:23398/2" value="100uF"/>
+<part name="C11" library="rcl" library_urn="urn:adsk.eagle:library:334" deviceset="CPOL-EU" device="153CLV-0605" package3d_urn="urn:adsk.eagle:package:23398/2" value="47uF">
+<spice>
+<pinmapping spiceprefix="C">
+<pinmap gate="G$1" pin="+" pinorder="1"/>
+<pinmap gate="G$1" pin="-" pinorder="2"/>
+</pinmapping>
+</spice>
+<attribute name="MPN" value="SC1E476M6L005VR"/>
+</part>
 <part name="GND15" library="supply1" library_urn="urn:adsk.eagle:library:371" deviceset="GND" device=""/>
 <part name="IC9" library="custom ICs" deviceset="RS422" device="-SO8" package3d_urn="urn:adsk.eagle:package:17511/1">
@@
 <part name="GND18" library="supply1" library_urn="urn:adsk.eagle:library:371" deviceset="GND" device=""/>
 <part name="R16" library="rcl" library_urn="urn:adsk.eagle:library:334" deviceset="R-EU_" device="R0805" package3d_urn="urn:adsk.eagle:package:23553/2" value="10K"/>
-<part name="IC12" library="custom ICs" deviceset="USBLC6-4" device="" package3d_urn="urn:adsk.eagle:package:30993/1"/>
+<part name="IC12" library="custom ICs" deviceset="USBLC6-4" device="" package3d_urn="urn:adsk.eagle:package:30993/1">
+<attribute name="MPN" value="USBLC6"/>
+</part>
 <part name="GND20" library="supply1" library_urn="urn:adsk.eagle:library:371" deviceset="GND" device=""/>
 <part name="R17" library="rcl" library_urn="urn:adsk.eagle:library:334" deviceset="R-EU_" device="R0805" package3d_urn="urn:adsk.eagle:package:23553/2" value="120R"/>
-<part name="S1" library="smd-special" library_urn="urn:adsk.eagle:library:362" deviceset="SWS006" device="" package3d_urn="urn:adsk.eagle:package:26472/1"/>
+<part name="S1" library="smd-special" library_urn="urn:adsk.eagle:library:362" deviceset="SWS006" device="" package3d_urn="urn:adsk.eagle:package:26472/1">
+<attribute name="MPN" value="A6S-6102-H"/>
+</part>
 <part name="R18" library="rcl" library_urn="urn:adsk.eagle:library:334" deviceset="R-EU_" device="R0805" package3d_urn="urn:adsk.eagle:package:23553/2" value="10K"/>
 <part name="R19" library="rcl" library_urn="urn:adsk.eagle:library:334" deviceset="R-EU_" device="R0805" package3d_urn="urn:adsk.eagle:package:23553/2" value="10K"/>
@@
 <part name="TRIG" library="custom connectors" deviceset="SMPAD-7" device=""/>
 <part name="GND22" library="supply1" library_urn="urn:adsk.eagle:library:371" deviceset="GND" device=""/>
-<part name="IC14" library="custom ICs" deviceset="74*1G157" device=""/>
+<part name="IC14" library="custom ICs" deviceset="74*1G157" device="">
+<attribute name="MPN" value="74LVC1G157GV.125"/>
+</part>
 <part name="C16" library="rcl" library_urn="urn:adsk.eagle:library:334" deviceset="C-EU" device="C0805" package3d_urn="urn:adsk.eagle:package:23617/2" value="100nF"/>
 <part name="H1" library="custom mounting" deviceset="HOLE" device="-3MM_PLATED"/>
@@
 <part name="H4" library="custom mounting" deviceset="HOLE" device="-3MM_PLATED"/>
 <part name="GND23" library="supply1" library_urn="urn:adsk.eagle:library:371" deviceset="GND" device=""/>
-<part name="Q1" library="custom passives" deviceset="RESONATOR_CRY" device="" value="16MHz"/>
+<part name="Q1" library="custom passives" deviceset="RESONATOR_CRY" device="" value="16MHz">
+<attribute name="MPN" value="3225-16M-SR"/>
+</part>
 <part name="C6" library="rcl" library_urn="urn:adsk.eagle:library:334" deviceset="C-EU" device="C0805" package3d_urn="urn:adsk.eagle:package:23617/2" value="100nF"/>
 <part name="GND24" library="supply1" library_urn="urn:adsk.eagle:library:371" deviceset="GND" device=""/>
@@
 <instance part="IC1" gate="A" x="58.42" y="101.6" smashed="yes" rot="R90">
 <attribute name="NAME" x="46.99" y="91.44" size="1.778" layer="95" rot="R90"/>
+<attribute name="MPN" x="58.42" y="101.6" size="1.778" layer="96" rot="R90" display="off"/>
 </instance>
 <instance part="C1" gate="G$1" x="25.4" y="22.86" smashed="yes">
@@
 <instance part="IC7" gate="A" x="271.78" y="53.34" smashed="yes">
 <attribute name="NAME" x="274.32" y="56.515" size="1.778" layer="95"/>
+<attribute name="MPN" x="271.78" y="53.34" size="1.778" layer="96" display="off"/>
 </instance>
 <instance part="IC7" gate="B" x="271.78" y="40.64" smashed="yes">
@@
 <attribute name="NAME" x="233.68" y="59.055" size="1.778" layer="95"/>
 <attribute name="VALUE" x="233.68" y="43.18" size="1.778" layer="96"/>
+<attribute name="MPN" x="241.3" y="53.34" size="1.778" layer="96" display="off"/>
 </instance>
 <instance part="IC8" gate="B" x="241.3" y="30.48" smashed="yes">
@@
 <attribute name="NAME" x="24.13" y="80.137" size="1.778" layer="95"/>
 <attribute name="VALUE" x="24.13" y="75.819" size="1.778" layer="96"/>
+<attribute name="MPN" x="27.94" y="78.74" size="1.778" layer="96" display="off"/>
 </instance>
 <instance part="C7" gate="G$1" x="71.12" y="22.86" smashed="yes">
@@
 <attribute name="NAME" x="36.703" y="69.0626" size="1.778" layer="95"/>
 <attribute name="VALUE" x="36.703" y="63.9826" size="1.778" layer="96"/>
+<attribute name="MPN" x="35.56" y="68.58" size="1.778" layer="96" display="off"/>
 </instance>
 <instance part="GND15" gate="1" x="35.56" y="58.42" smashed="yes">
@@
 <instance part="IC12" gate="A" x="302.26" y="193.04" smashed="yes" rot="R90">
 <attribute name="NAME" x="290.83" y="182.88" size="1.778" layer="95" rot="R90"/>
+<attribute name="MPN" x="302.26" y="193.04" size="1.778" layer="96" rot="R90" display="off"/>
 </instance>
 <instance part="GND20" gate="1" x="302.26" y="172.72" smashed="yes">
@@
 <instance part="S1" gate="G$1" x="271.78" y="175.26" smashed="yes">
 <attribute name="NAME" x="264.16" y="172.72" size="1.778" layer="95" rot="R90"/>
+<attribute name="MPN" x="271.78" y="175.26" size="1.778" layer="96" display="off"/>
 </instance>
 <instance part="R18" gate="G$1" x="279.4" y="198.12" smashed="yes" rot="R90">
@@
 <attribute name="NAME" x="233.68" y="114.935" size="1.778" layer="95"/>
 <attribute name="VALUE" x="233.68" y="96.52" size="1.778" layer="96"/>
+<attribute name="MPN" x="238.76" y="106.68" size="1.778" layer="96" display="off"/>
 </instance>
 <instance part="IC14" gate="P" x="142.24" y="22.86" smashed="yes">
@@
 <attribute name="NAME" x="27.94" y="181.61" size="1.778" layer="95" rot="R90"/>
 <attribute name="VALUE" x="34.798" y="179.07" size="1.778" layer="96" rot="R90"/>
+<attribute name="MPN" x="30.48" y="182.88" size="1.778" layer="96" rot="R90" display="off"/>
 </instance>
 <instance part="C6" gate="G$1" x="132.08" y="157.48" smashed="yes">
@@
 </segment>
 <segment>
-<pinref part="IC13" gate="IC" pin="PC5(ADC5/SCL/PCINT13)"/>
-<wire x1="63.5" y1="160.02" x2="38.1" y2="160.02" width="0.1524" layer="91"/>
-<label x="38.1" y="160.02" size="1.778" layer="95" rot="R180" xref="yes"/>
+<pinref part="IC13" gate="IC" pin="PD7(AIN1/PCINT23)"/>
+<wire x1="129.54" y1="177.8" x2="152.4" y2="177.8" width="0.1524" layer="91"/>
+<label x="152.4" y="177.8" size="1.778" layer="95" xref="yes"/>
 </segment>
 </net>
@@
 </sheet>
 </sheets>
+<errors>
+</errors>
 </schematic>
 </drawing>

Commit message: Timed trigger WIP
Connections:
- net B renamed L3
- net B+ renamed L3+
- net B- renamed L3-
- net G renamed L2
- net G+ renamed L2+
- net G- renamed L2-
- net R renamed L1
- net R+ renamed L1+
- net R- renamed L1-
Changed lines of the file:
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@@
 </segment>
 </net>
-<net name="R" class="0">
+<net name="L1" class="0">
 <segment>
 <pinref part="IC7" gate="A" pin="O"/>
@@
 </segment>
 </net>
-<net name="G" class="0">
+<net name="L2" class="0">
 <segment>
 <pinref part="IC7" gate="B" pin="O"/>
@@
 </segment>
 </net>
-<net name="B" class="0">
+<net name="L3" class="0">
 <segment>
 <pinref part="IC7" gate="C" pin="O"/>
@@
 </segment>
 </net>
-<net name="R+" class="0">
+<net name="L1+" class="0">
 <segment>
 <pinref part="IC9" gate="G$1" pin="D+"/>
@@
 </segment>
 </net>
-<net name="R-" class="0">
+<net name="L1-" class="0">
 <segment>
 <pinref part="IC9" gate="G$1" pin="D-"/>
@@
 </segment>
 </net>
-<net name="G+" class="0">
+<net name="L2+" class="0">
 <segment>
 <pinref part="IC10" gate="G$1" pin="D+"/>
@@
 </segment>
 </net>
-<net name="G-" class="0">
+<net name="L2-" class="0">
 <segment>
 <pinref part="IC10" gate="G$1" pin="D-"/>
@@
 </segment>
 </net>
-<net name="B+" class="0">
+<net name="L3+" class="0">
 <segment>
 <pinref part="IC11" gate="G$1" pin="D+"/>
@@
 </segment>
 </net>
-<net name="B-" class="0">
+<net name="L3-" class="0">
 <segment>
 <pinref part="IC11" gate="G$1" pin="D-"/>

Commit message: tweaks
Connections:
- net RGB_IN renamed L_IN
- net RGB_SEL0 renamed L_SEL0
- net RGB_SEL1 renamed L_SEL1
Changed lines of the file:
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@@
 </segment>
 </net>
-<net name="RGB_IN" class="0">
+<net name="L_IN" class="0">
 <segment>
 <pinref part="IC7" gate="D" pin="I1"/>
@@
 </segment>
 </net>
-<net name="RGB_SEL0" class="0">
+<net name="L_SEL0" class="0">
 <segment>
 <pinref part="IC8" gate="A" pin="A"/>
@@
 </segment>
 </net>
-<net name="RGB_SEL1" class="0">
+<net name="L_SEL1" class="0">
 <segment>
 <pinref part="IC8" gate="A" pin="B"/>
