File: PCB/HDR camera controller/HDR camera controller.sch (EAGLE design)
At the start: 63 parts, among them IC1 USBLC6-4, IC10 RS422-SO8, IC11 RS422-SO8, IC12 USBLC6-4, IC14 741G157, IC2 RS422-SO8, IC3 RS422-SO8, IC4 RS422-SO8, IC6 FT232RL, IC7 74HC00D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

Commit message: amogus did not print, got rid of it :(
Other:
- note added: "USB <-> UART"
- note removed: "USB <-> TTL"
Changed lines of the file:
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@@
 <wire x1="0" y1="134.62" x2="175.26" y2="134.62" width="0.254" layer="90"/>
 <wire x1="175.26" y1="134.62" x2="175.26" y2="43.18" width="0.254" layer="90"/>
-<wire x1="175.26" y1="43.18" x2="25.4" y2="43.18" width="0.254" layer="90"/>
-<text x="2.54" y="45.72" size="2.54" layer="90">USB &lt;-&gt; TTL</text>
-<wire x1="25.4" y1="43.18" x2="0" y2="43.18" width="0.254" layer="90"/>
-<wire x1="0" y1="50.8" x2="25.4" y2="50.8" width="0.254" layer="90"/>
-<wire x1="25.4" y1="50.8" x2="25.4" y2="43.18" width="0.254" layer="90"/>
+<wire x1="175.26" y1="43.18" x2="27.94" y2="43.18" width="0.254" layer="90"/>
+<text x="2.54" y="45.72" size="2.54" layer="90">USB &lt;-&gt; UART</text>
+<wire x1="27.94" y1="43.18" x2="0" y2="43.18" width="0.254" layer="90"/>
+<wire x1="0" y1="50.8" x2="27.94" y2="50.8" width="0.254" layer="90"/>
+<wire x1="27.94" y1="50.8" x2="27.94" y2="43.18" width="0.254" layer="90"/>
 <wire x1="302.26" y1="0" x2="302.26" y2="7.62" width="0.254" layer="90"/>
 <wire x1="302.26" y1="7.62" x2="302.26" y2="134.62" width="0.254" layer="90"/>

Commit message: EEPROM implemented and tested, PCB docs
Other:
- note removed: "Bypass"
- note removed: "HW trigger mux"
- note removed: "I/O connectors"
- note removed: "RGB demux"
- note removed: "RS422 drivers"
- note removed: "USB <-> UART"
