File: PCB/HDR camera controller/V1.1/HDR camera controller.sch (EAGLE design)
At the start: 63 parts, among them IC1 USBLC6-4, IC10 RS422-SO8, IC11 RS422-SO8, IC12 USBLC6-4, IC14 741G157, IC2 RS422-SO8, IC3 RS422-SO8, IC4 RS422-SO8, IC6 FT232RL, IC7 74HC00D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

Commit message: wip
Connections:
- net ENC_B: now also IC13IC.PD4(T0/XCK/PCINT20); no longer IC13IC.PC4(ADC4/SDA/PCINT12)
- net LINE_IN_1: now also IC13IC.PB1(OC1A/PCINT1); no longer IC13IC.PD6(AIN0/OC0A/PCINT22)
- net L_IN: now also IC13IC.PB2(SS/OC1B/PCINT2); no longer IC13IC.PD5(T1/OC0B/PCINT21)
Changed lines of the file:
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@@
 <net name="LINE_IN_1" class="0">
 <segment>
-<pinref part="IC13" gate="IC" pin="PD6(AIN0/OC0A/PCINT22)"/>
-<wire x1="165.1" y1="119.38" x2="167.64" y2="119.38" width="0.1524" layer="91"/>
-<label x="167.64" y="119.38" size="1.778" layer="95" xref="yes"/>
+<pinref part="IC13" gate="IC" pin="PB1(OC1A/PCINT1)"/>
+<wire x1="99.06" y1="132.08" x2="93.98" y2="132.08" width="0.1524" layer="91"/>
+<label x="93.98" y="132.08" size="1.778" layer="95" rot="R180" xref="yes"/>
 </segment>
 </net>
@@
 <net name="L_IN" class="0">
 <segment>
-<pinref part="IC13" gate="IC" pin="PD5(T1/OC0B/PCINT21)"/>
-<wire x1="165.1" y1="121.92" x2="187.96" y2="121.92" width="0.1524" layer="91"/>
-<label x="187.96" y="121.92" size="1.778" layer="95" xref="yes"/>
-</segment>
-<segment>
 <pinref part="IC7" gate="D" pin="I1"/>
 <wire x1="170.18" y1="50.8" x2="167.64" y2="50.8" width="0.1524" layer="91"/>
@@
 <junction x="167.64" y="50.8"/>
 <label x="165.1" y="50.8" size="1.778" layer="95" rot="R180" xref="yes"/>
+</segment>
+<segment>
+<pinref part="IC13" gate="IC" pin="PB2(SS/OC1B/PCINT2)"/>
+<wire x1="99.06" y1="129.54" x2="78.74" y2="129.54" width="0.1524" layer="91"/>
+<label x="78.74" y="129.54" size="1.778" layer="95" rot="R180" xref="yes"/>
 </segment>
 </net>
@@
 <net name="ENC_B" class="0">
 <segment>
-<pinref part="IC13" gate="IC" pin="PC4(ADC4/SDA/PCINT12)"/>
-<wire x1="99.06" y1="101.6" x2="93.98" y2="101.6" width="0.1524" layer="91"/>
-<label x="93.98" y="101.6" size="1.778" layer="95" rot="R180" xref="yes"/>
-</segment>
-<segment>
 <wire x1="91.44" y1="25.4" x2="91.44" y2="20.32" width="0.1524" layer="91"/>
 <wire x1="91.44" y1="20.32" x2="25.4" y2="20.32" width="0.1524" layer="91"/>
@@
 <pinref part="TRIG" gate="-3" pin="P"/>
 </segment>
+<segment>
+<pinref part="IC13" gate="IC" pin="PD4(T0/XCK/PCINT20)"/>
+<wire x1="165.1" y1="124.46" x2="167.64" y2="124.46" width="0.1524" layer="91"/>
+<label x="167.64" y="124.46" size="1.778" layer="95" xref="yes"/>
+</segment>
 </net>

Commit message: Line in 2 activation during 1st exposure
Connections:
- new net LINE_IN_2: IC13IC.PC5(ADC5/SCL/PCINT13), IC3G$1.DI
- new net LINE_IN_3: IC4G$1.DI
- net ENC_A: no longer IC3G$1.DI
- net ENC_B: no longer IC4G$1.DI
Changed lines of the file:
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@@
-</segment>
-</net>
-<net name="ENC_B" class="0">
-<segment>
-<pinref part="IC4" gate="G$1" pin="DI"/>
-<wire x1="78.74" y1="68.58" x2="73.66" y2="68.58" width="0.1524" layer="91"/>
-<label x="73.66" y="68.58" size="1.778" layer="95" rot="R180" xref="yes"/>
-</segment>
-</net>
-<net name="ENC_A" class="0">
-<segment>
-<pinref part="IC3" gate="G$1" pin="DI"/>
-<wire x1="78.74" y1="104.14" x2="73.66" y2="104.14" width="0.1524" layer="91"/>
-<label x="73.66" y="104.14" size="1.778" layer="95" rot="R180" xref="yes"/>
 </segment>
 </net>
@@
 <pinref part="IC11" gate="G$1" pin="R-"/>
 <wire x1="172.72" y1="50.8" x2="175.26" y2="50.8" width="0.1524" layer="91"/>
+</segment>
+</net>
+<net name="LINE_IN_2" class="0">
+<segment>
+<pinref part="IC3" gate="G$1" pin="DI"/>
+<wire x1="78.74" y1="104.14" x2="73.66" y2="104.14" width="0.1524" layer="91"/>
+<label x="73.66" y="104.14" size="1.778" layer="95" rot="R180" xref="yes"/>
+</segment>
+</net>
+<net name="LINE_IN_3" class="0">
+<segment>
+<pinref part="IC4" gate="G$1" pin="DI"/>
+<wire x1="78.74" y1="68.58" x2="73.66" y2="68.58" width="0.1524" layer="91"/>
+<label x="73.66" y="68.58" size="1.778" layer="95" rot="R180" xref="yes"/>
 </segment>
 </net>
@@
 </segment>
 </net>
+<net name="LINE_IN_2" class="0">
+<segment>
+<pinref part="IC13" gate="IC" pin="PC5(ADC5/SCL/PCINT13)"/>
+<wire x1="99.06" y1="99.06" x2="73.66" y2="99.06" width="0.1524" layer="91"/>
+<label x="73.66" y="99.06" size="1.778" layer="95" rot="R180" xref="yes"/>
+</segment>
+</net>

Commit message: Documentation
Parts:
- added R6: 10K, rcl:R-EU_R0805
Connections:
- net GND: now also R6.1
- net LINE_IN_3: now also R6.2
Changed lines of the file:
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@@
 <layer number="202" name="bNamesOnPCB" color="3" fill="1" visible="yes" active="yes"/>
 </layers>
-<schematic xreflabel="%F%N" xrefpart="/%S.%C%R">
+<schematic xreflabel="%F%N" xrefpart="/">
 <attributes>
 </attributes>
@@
 <part name="FRAME2" library="frames" library_urn="urn:adsk.eagle:library:229" deviceset="A4L-LOC" device=""/>
 <part name="FRAME3" library="frames" library_urn="urn:adsk.eagle:library:229" deviceset="A4L-LOC" device=""/>
+<part name="R6" library="rcl" library_urn="urn:adsk.eagle:library:334" deviceset="R-EU_" device="R0805" package3d_urn="urn:adsk.eagle:package:23553/2" value="10K"/>
+<part name="GND25" library="supply1" library_urn="urn:adsk.eagle:library:371" deviceset="GND" device=""/>
 </parts>
 <sheets>
@@
 <attribute name="VALUE" x="183.642" y="49.53" size="1.778" layer="96" rot="R90"/>
 </instance>
+<instance part="R6" gate="G$1" x="76.2" y="60.96" smashed="yes" rot="R90">
+<attribute name="NAME" x="74.7014" y="57.15" size="1.778" layer="95" rot="R90"/>
+<attribute name="VALUE" x="79.502" y="57.15" size="1.778" layer="96" rot="R90"/>
+</instance>
+<instance part="GND25" gate="1" x="76.2" y="48.26" smashed="yes">
+<attribute name="VALUE" x="73.66" y="45.72" size="1.778" layer="96"/>
+</instance>
 </instances>
 <busses>
@@
 <pinref part="GND21" gate="1" pin="GND"/>
 <wire x1="104.14" y1="50.8" x2="101.6" y2="50.8" width="0.1524" layer="91"/>
+</segment>
+<segment>
+<pinref part="GND25" gate="1" pin="GND"/>
+<pinref part="R6" gate="G$1" pin="1"/>
+<wire x1="76.2" y1="50.8" x2="76.2" y2="55.88" width="0.1524" layer="91"/>
 </segment>
 </net>
@@
 <segment>
 <pinref part="IC4" gate="G$1" pin="DI"/>
-<wire x1="78.74" y1="68.58" x2="73.66" y2="68.58" width="0.1524" layer="91"/>
+<wire x1="78.74" y1="68.58" x2="76.2" y2="68.58" width="0.1524" layer="91"/>
 <label x="73.66" y="68.58" size="1.778" layer="95" rot="R180" xref="yes"/>
-</segment>
-</net>
+<pinref part="R6" gate="G$1" pin="2"/>
+<wire x1="76.2" y1="68.58" x2="73.66" y2="68.58" width="0.1524" layer="91"/>
+<wire x1="76.2" y1="66.04" x2="76.2" y2="68.58" width="0.1524" layer="91"/>
+<junction x="76.2" y="68.58"/>
+</segment>
+</net>
